Commit message: added Gazebo model

File: src/urdf_example-main/src/description/my_example_robot_v2.urdf.xacro (robot description, xacro)
@@ -4,25 +4,35 @@
     <!-- As we move through the file, new things to note will be pointed out. -->
     <!-- It's not meant an example of GOOD design, but an example of some of the various features of URDF/xacro. -->
-    <xacro:property name="box_x" value="0.54" />
-    <xacro:property name="box_y" value="0.925" />
+    <xacro:property name="box_y" value="0.54" />
+    <xacro:property name="box_x" value="0.925" />
     <xacro:property name="box_z" value="0.304" />
     <xacro:property name="box_m" value="100" />
     <xacro:property name="box_off_z" value="0.484" />
-    <xacro:property name="cyl_l" value="0.05" />
+    <xacro:property name="cyl_l" value="0.1" />
     <xacro:property name="cyl_r" value="0.28" />
     <xacro:property name="cyl_m" value="10" />
     <xacro:property name="cyl_off_x" value="0.3068" />
     <xacro:property name="cyl_off_y" value="0.3425" />
-    <xacro:property name="cyl_off_z" value="-0.204" />
+    <xacro:property name="cyl_off_z" value="${box_off_z-0.204}" />
     <xacro:property name="rot_90" value="${pi/2}" />
     <!-- This will include all the contents of example_include.xacro first. Go check it out! -->
     <xacro:include filename="example_include.xacro" />
     <!-- This first link called "world" is empty -->
-    <link name="world"></link>
+    <!-- <link name="world"></link> -->
+    <link name="dummy"></link>
+    <!-- <joint name="world_joint" type="fixed">
+        <parent link="world"/>
+        <child link="body_link" />
+    </joint> -->
     <!-- A simple fixed joint from our empty world link, to our base. -->
     <!-- The base origin is offset from the world origin. -->
+    <!-- <joint name="chassis_joint" type="fixed"> -->
+        <!-- <origin xyz="0 0 ${box_off_z}" rpy="0 0 0"/> -->
+        <!-- <parent link="world"/> -->
+        <!-- <child link="chassis_link"/>         -->
+    <!-- </joint> -->
     <joint name="chassis_joint" type="fixed">
-        <origin xyz="0 0 ${box_off_z}" rpy="0 0 0"/>
-        <parent link="world"/>
+        <!-- <origin xyz="0 0 ${box_off_z}" rpy="0 0 0"/> -->
+        <parent link="dummy"/>
         <child link="chassis_link"/>
     </joint>
@@ -37,7 +47,11 @@
     <!-- - We specified the colour manually (but still need to enter a name) -->
     <!-- - We specified all the inertial parameters manually -->
+    <!-- ##############################################  -->
+    <!-- Chassis Link  -->
+    <!-- ##############################################  -->
     <link name="chassis_link">
         <visual>
-            <origin xyz="0 0 ${-box_z/2}" rpy="0 0 0"/>
+            <origin xyz="0 0 ${box_off_z-box_z/2}" rpy="0 0 0"/>
+            <!-- <origin xyz="0 0 ${box_z}" rpy="0 0 0"/> -->
             <geometry>
                 <box size="${box_x} ${box_y} ${box_z}" />
@@ -46,5 +60,6 @@
         </visual>
         <collision>
-            <origin xyz="0 0 ${-box_z/2}" rpy="0 0 0"/>
+            <origin xyz="0 0 ${box_off_z-box_z/2}" rpy="0 0 0"/>
+            <!-- <origin xyz="0 0 ${box_z}" rpy="0 0 0"/> -->
             <geometry>
                 <box size="${box_x} ${box_y} ${box_z}" />
@@ -52,13 +67,18 @@
         </collision>
        <xacro:inertial_box mass="${box_m}" x="${box_x}" y="${box_y}" z="${box_z}">
-            <origin xyz="0.0 0 ${-box_z/2}" rpy="0 0 0"/>
+            <origin xyz="0.0 0 ${box_off_z-box_z/2}" rpy="0 0 0"/>
+            <!-- <origin xyz="0 0 ${box_z}" rpy="0 0 0"/> -->
         </xacro:inertial_box>
     </link>
+    <!-- ##############################################  -->
     <!-- WHEEL 1  +x +y-->
-    <!--  -->
-    <joint name="wheel_1_joint" type="fixed">
-        <origin xyz="${cyl_off_x} ${cyl_off_y} ${cyl_off_z}" rpy="0 ${rot_90} 0"/>
+    <!-- ##############################################  -->
+    <joint name="wheel_1_joint" type="continuous">
+        <origin xyz="${cyl_off_x} ${cyl_off_y} ${cyl_off_z}" rpy="${rot_90} 0 0"/>
         <parent link="chassis_link"/>
         <child link="wheel_1_link"/>
+        <axis xyz="0 0 1" />
+        <limit effort="1000" velocity="1000"/>
+        <dynamics damping="1.0" friction="1.0"/>
     </joint>
     <link name="wheel_1_link">
@@ -80,10 +100,14 @@
         </xacro:inertial_cylinder>
     </link>
+    <!-- ##############################################  -->
     <!-- WHEEL 2  +x -y -->
-    <!--  -->
-    <joint name="wheel_2_joint" type="fixed">
-        <origin xyz="${cyl_off_x} ${-cyl_off_y} ${cyl_off_z}" rpy="0 ${rot_90} 0"/>
+    <!-- ##############################################  -->
+    <joint name="wheel_2_joint" type="continuous">
+        <origin xyz="${cyl_off_x} ${-cyl_off_y} ${cyl_off_z}" rpy="${rot_90} 0 0"/>
         <parent link="chassis_link"/>
         <child link="wheel_2_link"/>
+        <axis xyz="0 0 1" />
+        <limit effort="1000" velocity="1000"/>
+        <dynamics damping="1.0" friction="1.0"/>
     </joint>
     <link name="wheel_2_link">
@@ -105,10 +129,14 @@
         </xacro:inertial_cylinder>
     </link>
+    <!-- ##############################################  -->
     <!-- WHEEL 3  -x -y -->
-    <!--  -->
-    <joint name="wheel_3_joint" type="fixed">
-        <origin xyz="${-cyl_off_x} ${-cyl_off_y} ${cyl_off_z}" rpy="0 ${rot_90} 0"/>
+    <!-- ##############################################  -->
+    <joint name="wheel_3_joint" type="continuous">
+        <origin xyz="${-cyl_off_x} ${-cyl_off_y} ${cyl_off_z}" rpy="${rot_90} 0 0"/>
         <parent link="chassis_link"/>
         <child link="wheel_3_link"/>
+        <axis xyz="0 0 1" />
+        <limit effort="1000" velocity="1000"/>
+        <dynamics damping="1.0" friction="1.0"/>
     </joint>
     <link name="wheel_3_link">
@@ -130,10 +158,14 @@
         </xacro:inertial_cylinder>
     </link>
+    <!-- ##############################################  -->
     <!-- WHEEL 4  -x +y -->
-    <!--  -->
-    <joint name="wheel_4_joint" type="fixed">
-        <origin xyz="${-cyl_off_x} ${cyl_off_y} ${cyl_off_z}" rpy="0 ${rot_90} 0"/>
+    <!-- ##############################################  -->
+    <joint name="wheel_4_joint" type="continuous">
+        <origin xyz="${-cyl_off_x} ${cyl_off_y} ${cyl_off_z}" rpy="${rot_90} 0 0"/>
         <parent link="chassis_link"/>
         <child link="wheel_4_link"/>
+        <axis xyz="0 0 1" />
+        <limit effort="1000" velocity="1000"/>
+        <dynamics damping="1.0" friction="1.0"/>
     </joint>
     <link name="wheel_4_link">
@@ -155,4 +187,4 @@
         </xacro:inertial_cylinder>
     </link>
-    <!-- <xacro:include filename="example_gazebo.xacro" /> -->
+    <xacro:include filename="my_example_gazebo.xacro" />
 </robot>
