Commit message: Backup

File: install/RobuROC_sim/share/RobuROC_sim/description/robot/RobuROC_gazebo.urdf.xacro (robot description, xacro)
@@ -17,4 +17,9 @@
     <xacro:property name="rot_90" value="${pi/2}" />
     <xacro:property name="max_vel" value="2" />
+    <xacro:property name="IMU_y" value="0.06" />
+    <xacro:property name="IMU_x" value="0.05" />
+    <xacro:property name="IMU_z" value="0.02" />
+    <xacro:property name="IMU_m" value="0.1" />
+    <xacro:property name="IMU_off_z" value="${0.484+IMU_z/2}" />
     <!-- This will include inertia and color functions -->
     <xacro:include filename="include_RobuROC.xacro" />
@@ -167,4 +172,30 @@
         </xacro:inertial_cylinder>
     </link>
+    <!-- ##############################################  -->
+    <!--                IMU                              -->
+    <!-- ##############################################  -->
+    <joint name="IMU_joint" type="fixed">
+        <origin xyz="0 0 ${IMU_off_z}"/>
+        <parent link="chassis_link"/>
+        <child link="IMU_link"/>
+    </joint>
+    <link name="IMU_link">
+        <visual>
+            <origin xyz="0 0 0" rpy="0 0 0"/>
+            <geometry>
+                <box size="${IMU_x} ${IMU_y} ${IMU_z}"/>
+            </geometry>
+            <material name="red" />
+        </visual>
+        <collision>
+            <origin xyz="0 0 0" rpy="0 0 0"/>
+            <geometry>
+                <box size="${IMU_x} ${IMU_y} ${IMU_z}" />
+            </geometry>
+        </collision>
+        <xacro:inertial_box mass="${IMU_m}" x="${IMU_x}" y="${IMU_y}" z="${IMU_z}">
+            <origin xyz="0.0 0 0" rpy="0 0 0"/>
+        </xacro:inertial_box>
+    </link>
     <!-- Include gazebo model -->
     <xacro:include filename="RobuROC_gazebo_sim.xacro" />

File: install/RobuROC_sim/share/RobuROC_sim/description/robot/RobuROC_gazebo_sim.xacro (robot description, xacro)
@@ -7,27 +7,34 @@
         <mu1> 0.2 </mu1>
         <mu2> 0.2 </mu2>
-        <material>Gazebo/Blue</material>
+        <material>Gazebo/Grey</material>
     </gazebo>
     <gazebo reference="wheel_1_link">
         <mu1> 0.2 </mu1>
         <mu2> 0.2 </mu2>
-        <material>Gazebo/Orange</material>
+        <material>Gazebo/Black</material>
     </gazebo>
     <gazebo reference="wheel_2_link">
         <mu1> 0.2 </mu1>
         <mu2> 0.2 </mu2>
-        <material>Gazebo/Orange</material>
+        <material>Gazebo/Black</material>
     </gazebo>
     <gazebo reference="wheel_3_link">
         <mu1> 0.2 </mu1>
         <mu2> 0.2 </mu2>
-        <material>Gazebo/Orange</material>
+        <material>Gazebo/Black</material>
     </gazebo>
     <gazebo reference="wheel_4_link">
         <mu1> 0.2 </mu1>
         <mu2> 0.2 </mu2>
-        <material>Gazebo/Orange</material>
+        <material>Gazebo/Black</material>
     </gazebo>
-<!-- Controller -->
+    <gazebo reference="IMU_link">
+        <mu1> 0.2 </mu1>
+        <mu2> 0.2 </mu2>
+        <material>Gazebo/Red</material>
+    </gazebo>
+<!-- #################################################################################### -->
+<!--                                Differential drive                                    -->
+<!-- #################################################################################### -->
     <gazebo>
         <!-- Gazebo plugin for differential drive -->
@@ -59,4 +66,7 @@
         </plugin>
     </gazebo>
+<!-- #################################################################################### -->
+<!--                                        IMU                                           -->
+<!-- #################################################################################### -->
     <!-- Gazebo requires the use of plugins to interact with other systems such as ROS. -->
     <!-- This plugin will publish the joint_states for the selected joints

File: install/RobuROC_sim/share/RobuROC_sim/description/robot/RobuROC_rviz_blocks.urdf.xacro (robot description, xacro)
@@ -17,12 +17,17 @@
     <xacro:property name="rot_90" value="${pi/2}" />
     <xacro:property name="max_vel" value="2" />
+    <xacro:property name="IMU_y" value="0.06" />
+    <xacro:property name="IMU_x" value="0.05" />
+    <xacro:property name="IMU_z" value="0.02" />
+    <xacro:property name="IMU_m" value="0.1" />
+    <xacro:property name="IMU_off_z" value="${IMU_z/2}" />
     <!-- This will include inertia and color functions -->
     <xacro:include filename="include_RobuROC.xacro" />
     <!-- Initial link is empty link called world -->
-    <link name="world"></link>
+    <link name="dummy"></link>
     <!-- Chassis joint has been off seted in z axis and set to fixed-->
     <joint name="chassis_joint" type="fixed">
-        <origin xyz="0 0 ${box_off_z}" rpy="0 0 0"/>
-        <parent link="world"/>
+        <!-- <origin xyz="0 0 ${box_off_z}" rpy="0 0 0"/> -->
+        <parent link="dummy"/>
         <child link="chassis_link"/>
     </joint>
@@ -165,4 +170,30 @@
         </xacro:inertial_cylinder>
     </link>
+    <!-- ##############################################  -->
+    <!--                IMU                              -->
+    <!-- ##############################################  -->
+    <joint name="IMU_joint" type="fixed">
+        <origin xyz="0 0 ${IMU_off_z}"/>
+        <parent link="chassis_link"/>
+        <child link="IMU_link"/>
+    </joint>
+    <link name="IMU_link">
+        <visual>
+            <origin xyz="0 0 0" rpy="0 0 0"/>
+            <geometry>
+                <box size="${IMU_x} ${IMU_y} ${IMU_z}"/>
+            </geometry>
+            <material name="red" />
+        </visual>
+        <collision>
+            <origin xyz="0 0 0" rpy="0 0 0"/>
+            <geometry>
+                <box size="${IMU_x} ${IMU_y} ${IMU_z}" />
+            </geometry>
+        </collision>
+        <xacro:inertial_box mass="${IMU_m}" x="${IMU_x}" y="${IMU_y}" z="${IMU_z}">
+            <origin xyz="0.0 0 0" rpy="0 0 0"/>
+        </xacro:inertial_box>
+    </link>
     <!-- Include gazebo model -->
     <xacro:include filename="RobuROC_gazebo_sim.xacro" />

File: install/RobuROC_sim/share/RobuROC_sim/description/robot/RobuROC_rviz_stl.urdf.xacro (robot description, xacro)
@@ -35,12 +35,11 @@
     <link name="chassis_link">
         <visual>
-            <origin xyz="0 0 0" rpy="${rot_90} 0 0"/>
+            <origin xyz="0 0 0" rpy="${rot_90} 0 ${rot_90}"/>
             <geometry>
-                <mesh filename="file://$(find RobuROC_sim)/meshes/chassis_SI.STL" scale = "${scale}"/>
+                <mesh filename="file://$(find RobuROC_sim)/meshes/chassis.STL" scale = "${scale}"/>
             </geometry>
             <material name="blue" />
         </visual>
         <collision>
-            <!-- <origin xyz="0 0 ${box_off_z-box_z/2}" rpy="0 0 0"/> -->
             <origin xyz="0 0 ${box_z}" rpy="0 0 0"/>
             <geometry>
@@ -50,5 +49,4 @@
        <xacro:inertial_box mass="${box_m}" x="${box_x}" y="${box_y}" z="${box_z}">
             <origin xyz="0.0 0 ${box_off_z-box_z/2}" rpy="0 0 0"/>
-            <!-- <origin xyz="0 0 ${box_z}" rpy="0 0 0"/> -->
         </xacro:inertial_box>
     </link>
@@ -67,8 +65,7 @@
     <link name="wheel_1_link">
         <visual>
-            <origin xyz="0 0 0" rpy="0 0 0"/>
+            <origin xyz="0 0 0" rpy="0 ${rot_90} 0"/>
             <geometry>
-                <!-- <cylinder length="${cyl_l}" radius="${cyl_r}" /> -->
-                <mesh filename="file://$(find RobuROC_sim)/meshes/wheel_SI.STL"/>
+                <mesh filename="file://$(find RobuROC_sim)/meshes/wheel.STL" scale="${scale}"/>
             </geometry>
             <material name="orange" />
@@ -97,8 +94,7 @@
     <link name="wheel_2_link">
         <visual>
-            <origin xyz="0 0 0" rpy="0 0 0"/>
+            <origin xyz="0 0 0" rpy="0 ${rot_90} 0"/>
             <geometry>
-                <!-- <cylinder length="${cyl_l}" radius="${cyl_r}" /> -->
-                <mesh filename="file://$(find RobuROC_sim)/meshes/wheel_SI.STL"/>
+                <mesh filename="file://$(find RobuROC_sim)/meshes/wheel.STL" scale="${scale}"/>
             </geometry>
             <material name="orange" />
@@ -127,8 +123,7 @@
     <link name="wheel_3_link">
         <visual>
-            <origin xyz="0 0 0" rpy="0 0 0"/>
+            <origin xyz="0 0 0" rpy="0 ${rot_90} 0"/>
             <geometry>
-                <!-- <cylinder length="${cyl_l}" radius="${cyl_r}" /> -->
-                <mesh filename="file://$(find RobuROC_sim)/meshes/wheel_SI.STL"/>
+                <mesh filename="file://$(find RobuROC_sim)/meshes/wheel.STL" scale="${scale}"/>
             </geometry>
             <material name="orange" />
@@ -157,8 +152,7 @@
     <link name="wheel_4_link">
         <visual>
-            <origin xyz="0 0 0" rpy="0 0 0"/>
+            <origin xyz="0 0 0" rpy="0 ${rot_90} 0"/>
             <geometry>
-                <!-- <cylinder length="${cyl_l}" radius="${cyl_r}" /> -->
-                <mesh filename="file://$(find RobuROC_sim)/meshes/wheel_SI.STL"/>
+                <mesh filename="file://$(find RobuROC_sim)/meshes/wheel.STL" scale="${scale}"/>
             </geometry>
             <material name="orange" />

File: install/RobuROC_sim/share/RobuROC_sim/description/robot/include_RobuROC.xacro (robot description, xacro)
@@ -14,4 +14,13 @@
     <material name="green">
         <color rgba="0.2 1 0.2 1"/>
+    </material>
+    <material name="red">
+        <color rgba="1 0.2 0.2 1"/>
+    </material>
+    <material name="black">
+        <color rgba="0 0 0 1"/>
+    </material>
+    <material name="grey">
+        <color rgba="0.5 0.5 0.5 1"/>
     </material>
     <!-- Specify some standard inertial calculations https://en.wikipedia.org/wiki/List_of_moments_of_inertia -->
