Commit message: Fixed realsense_plugin, added velodyne rtab launch

File: src/RobuROC_sim/src/description/RobuROC_core.urdf.xacro (robot description, xacro)
@@ -5,4 +5,13 @@
     <!-- Initial link is empty link called base_link -->
     <link name="base_link"></link>
+    <!-- BASE_FOOTPRINT LINK -->
+    <!-- link for SLAM -->
+    <joint name="base_footprint_joint" type="fixed">
+        <parent link="base_link"/>
+        <child link="base_footprint"/>
+        <origin xyz="0 0 0" rpy="0 0 0"/>
+    </joint>
+    <link name="base_footprint">
+    </link>
     <!-- ##############################################  -->
     <!--                Chassis Link                     -->

File: src/RobuROC_sim/src/description/RobuROC_model.urdf.xacro (robot description, xacro)
@@ -10,4 +10,5 @@
     <!-- Add Lidar velodyne-16 -->
     <xacro:include filename="lidar_vlp_16.xacro" />
+    <!-- <xacro:include filename="lidar.xacro"/> -->
     <!-- Include gazebo model -->
     <xacro:include filename="RobuROC_gazebo_sim.xacro" />

File: src/RobuROC_sim/src/description/VLP-16.urdf.xacro (robot description, xacro)
@@ -84,5 +84,15 @@
             </noise>
           </ray>
+          <!-- <plugin name="laser_controller" filename="libgazebo_ros_ray_sensor.so"> -->
+            <!-- <ros> -->
+              <!-- <argument>~/out:=scan</argument> -->
+            <!-- </ros> -->
+            <!-- <output_type>sensor_msgs/LaserScan</output_type> -->
+            <!-- <frame_name>${name}</frame_name> -->
+          <!-- </plugin> -->
           <plugin name="gazebo_ros_laser_controller" filename="libgazebo_ros_velodyne_laser.so">
+            <ros>
+              <argument>~/out:=scan</argument>
+            </ros>
             <topicName>${topic}</topicName>
             <frameName>${name}</frameName>

File: src/RobuROC_sim/src/description/_d435.gazebo.xacro (robot description, xacro)
@@ -9,7 +9,4 @@
     <!-- Load parameters to model's main link-->
     <xacro:property name="deg_to_rad" value="0.01745329251994329577" />
-    <!-- ##############################################  -->
-    <!--                RGB camera                       -->
-    <!-- ##############################################  -->
     <gazebo reference="${reference_link}">
       <self_collide>0</self_collide>
@@ -47,26 +44,5 @@
         <update_rate>30</update_rate>
         <visualize>1</visualize>
-            <plugin name="${topics_ns}camera" filename="libgazebo_ros_camera.so">
-                <frame_name>${color_optical_frame}</frame_name>
-            </plugin>
-        </sensor>
-    </gazebo>
-    <!-- ##############################################  -->
-    <!--                Infrared camera 1                -->
-    <!-- ##############################################  -->
-    <gazebo reference="${reference_link}">
-      <self_collide>0</self_collide>
-      <enable_wind>0</enable_wind>
-      <kinematic>0</kinematic>
-      <gravity>1</gravity>
-      <!--<mu>1</mu>-->
-      <mu2>1</mu2>
-      <fdir1>0 0 0</fdir1>
-      <!--<slip1>0</slip1>
-      <slip2>0</slip2>-->
-      <kp>1e+13</kp>
-      <kd>1</kd>
-      <!--<max_vel>0.01</max_vel>
-      <min_depth>0</min_depth>-->
+      </sensor>
       <sensor name="${camera_name}ired1" type="camera">
         <camera name="${camera_name}">
@@ -90,26 +66,5 @@
         <update_rate>90</update_rate>
         <visualize>0</visualize>
-            <plugin name="${topics_ns}infra1" filename="libgazebo_ros_camera.so">
-                <frame_name>${infrared1_optical_frame}</frame_name>
-            </plugin>
-        </sensor>
-    </gazebo>
-    <!-- ##############################################  -->
-    <!--                Infrared camera 2                -->
-    <!-- ##############################################  -->
-    <gazebo reference="${reference_link}">
-      <self_collide>0</self_collide>
-      <enable_wind>0</enable_wind>
-      <kinematic>0</kinematic>
-      <gravity>1</gravity>
-      <!--<mu>1</mu>-->
-      <mu2>1</mu2>
-      <fdir1>0 0 0</fdir1>
-      <!--<slip1>0</slip1>
-      <slip2>0</slip2>-->
-      <kp>1e+13</kp>
-      <kd>1</kd>
-      <!--<max_vel>0.01</max_vel>
-      <min_depth>0</min_depth>-->
+      </sensor>
       <sensor name="${camera_name}ired2" type="camera">
         <camera name="${camera_name}">
@@ -133,13 +88,5 @@
         <update_rate>90</update_rate>
         <visualize>0</visualize>
-            <plugin name="${topics_ns}infra2" filename="libgazebo_ros_camera.so">
-                <frame_name>${infrared2_optical_frame}</frame_name>
-            </plugin>
-        </sensor>
-    </gazebo>
-    <!-- ##############################################  -->
-    <!--               Depth camera 2                    -->
-    <!-- ##############################################  -->
-    <gazebo reference="${reference_link}">
+      </sensor>
       <sensor name="${camera_name}depth" type="depth">
         <camera name="${camera_name}">
@@ -162,37 +109,32 @@
         <update_rate>90</update_rate>
         <visualize>0</visualize>
-          <plugin name="${topics_ns}depth" filename="libgazebo_ros_camera.so">
-            <frame_name>${depth_optical_frame}</frame_name>
-            <min_depth>0.2</min_depth>
-            <max_depth>10.0</max_depth>
-          </plugin>
       </sensor>
     </gazebo>
-    <!-- <gazebo> -->
-      <!-- <plugin name="${topics_ns}" filename="librealsense_gazebo_plugin.so"> -->
-        <!-- <prefix>${camera_name}</prefix> -->
-        <!-- <depthUpdateRate>30.0</depthUpdateRate> -->
-        <!-- <colorUpdateRate>30.0</colorUpdateRate> -->
-        <!-- <infraredUpdateRate>30.0</infraredUpdateRate> -->
-        <!-- <depthTopicName>depth/image_raw</depthTopicName> -->
-        <!-- <depthCameraInfoTopicName>depth/camera_info</depthCameraInfoTopicName> -->
-        <!-- <colorTopicName>color/image_raw</colorTopicName> -->
-        <!-- <colorCameraInfoTopicName>color/camera_info</colorCameraInfoTopicName> -->
-        <!-- <infrared1TopicName>infra1/image_raw</infrared1TopicName> -->
-        <!-- <infrared1CameraInfoTopicName>infra1/camera_info</infrared1CameraInfoTopicName> -->
-        <!-- <infrared2TopicName>infra2/image_raw</infrared2TopicName> -->
-        <!-- <infrared2CameraInfoTopicName>infra2/camera_info</infrared2CameraInfoTopicName> -->
-        <!-- <colorOpticalframeName>${color_optical_frame}</colorOpticalframeName> -->
-        <!-- <depthOpticalframeName>${depth_optical_frame}</depthOpticalframeName> -->
-        <!-- <infrared1OpticalframeName>${infrared1_optical_frame}</infrared1OpticalframeName> -->
-        <!-- <infrared2OpticalframeName>${infrared2_optical_frame}</infrared2OpticalframeName> -->
-        <!-- <rangeMinDepth>0.2</rangeMinDepth> -->
-        <!-- <rangeMaxDepth>10.0</rangeMaxDepth> -->
-        <!-- <pointCloud>${publish_pointcloud}</pointCloud> -->
-        <!-- <pointCloudTopicName>depth/color/points</pointCloudTopicName> -->
-        <!-- <pointCloudCutoff>0.25</pointCloudCutoff> -->
-        <!-- <pointCloudCutoffMax>9.0</pointCloudCutoffMax> -->
-      <!-- </plugin> -->
-    <!-- </gazebo> -->
+    <gazebo>
+      <plugin name="${topics_ns}" filename="librealsense_gazebo_plugin.so">
+        <prefix>${camera_name}</prefix>
+        <depthUpdateRate>30.0</depthUpdateRate>
+        <colorUpdateRate>30.0</colorUpdateRate>
+        <infraredUpdateRate>30.0</infraredUpdateRate>
+        <depthTopicName>${topics_ns}/depth/image_raw</depthTopicName>
+        <depthCameraInfoTopicName>${topics_ns}/depth/camera_info</depthCameraInfoTopicName>
+        <colorTopicName>${topics_ns}/color/image_raw</colorTopicName>
+        <colorCameraInfoTopicName>${topics_ns}/color/camera_info</colorCameraInfoTopicName>
+        <infrared1TopicName>${topics_ns}/infra1/image_raw</infrared1TopicName>
+        <infrared1CameraInfoTopicName>${topics_ns}/infra1/camera_info</infrared1CameraInfoTopicName>
+        <infrared2TopicName>${topics_ns}/infra2/image_raw</infrared2TopicName>
+        <infrared2CameraInfoTopicName>${topics_ns}/infra2/camera_info</infrared2CameraInfoTopicName>
+        <colorOpticalframeName>${color_optical_frame}</colorOpticalframeName>
+        <depthOpticalframeName>${depth_optical_frame}</depthOpticalframeName>
+        <infrared1OpticalframeName>${infrared1_optical_frame}</infrared1OpticalframeName>
+        <infrared2OpticalframeName>${infrared2_optical_frame}</infrared2OpticalframeName>
+        <rangeMinDepth>0.2</rangeMinDepth>
+        <rangeMaxDepth>10.0</rangeMaxDepth>
+        <pointCloud>${publish_pointcloud}</pointCloud>
+        <pointCloudTopicName>${topics_ns}/depth/color/points</pointCloudTopicName>
+        <pointCloudCutoff>0.25</pointCloudCutoff>
+        <pointCloudCutoffMax>9.0</pointCloudCutoffMax>
+      </plugin>
+    </gazebo>
   </xacro:macro>
 </robot>

File: src/RobuROC_sim/src/description/lidar.xacro (robot description, xacro)
@@ -2,7 +2,7 @@
 <robot xmlns:xacro="http://www.ros.org/wiki/xacro" >
     <joint name="laser_joint" type="fixed">
-        <parent link="chassis"/>
+        <parent link="base_link"/>
         <child link="laser_frame"/>
-        <origin xyz="0.122 0 0.212" rpy="0 0 0"/>
+        <origin xyz="0.122 0 0.5" rpy="0 0 0"/>
     </joint>
     <link name="laser_frame">
@@ -52,5 +52,5 @@
                     <argument>~/out:=scan</argument>
                 </ros>
-                <output_type>sensor_msgs/LaserScan</output_type>
+                <output_type>sensor_msgs/PointCloud2</output_type>
                 <frame_name>laser_frame</frame_name>
             </plugin>

File: src/RobuROC_sim/src/description/lidar_vlp_16.xacro (robot description, xacro)
@@ -4,5 +4,5 @@
   <xacro:property name="gpu" value="$(arg gpu)" />
   <xacro:include filename="VLP-16.urdf.xacro" />
-  <xacro:VLP-16 parent="base_link" name="velodyne" topic="velodyne_points" hz="10" samples="440" gpu="${gpu}">
+  <xacro:VLP-16 parent="base_link" name="velodyne" topic="/velodyne_points" hz="10" samples="440" gpu="${gpu}">
     <origin xyz="${lidar_origin}" rpy="0 0 0" />
   </xacro:VLP-16>
