Commit message: Fixed velodyne and camera launch, cameras has to be calibrated

File: src/RobuROC_sim/src/description/include_RobuROC.xacro (robot description, xacro)
@@ -45,5 +45,5 @@
     <!--                    Lidar                  -->
     <!-- ######################################### -->
-    <xacro:property name="lidar_off_x" value="0.12" />
+    <xacro:property name="lidar_off_x" value="-0.12" />
     <xacro:property name="lidar_off_z" value="${box_off_z+0.155}" />
     <xacro:property name="lidar_origin" value="${lidar_off_x} 0 ${lidar_off_z}" />

Commit message: Calibrated cameras, RTAB map based on Lidar ready for test

File: src/RobuROC_sim/src/description/include_RobuROC.xacro (robot description, xacro)
@@ -36,5 +36,5 @@
     <!-- ######################################### -->
     <xacro:property name="camera_off_x" value="0.6" />
-    <xacro:property name="camera_off_z" value="0.45" />
+    <xacro:property name="camera_off_z" value="0.55" />
     <xacro:property name="camera_rot" value="${16*pi/180}" />
     <xacro:property name="camera_1_origin" value="${camera_off_x} 0 ${camera_off_z}" />
