Commit message: Updated for minor issues related to control and Rtabmap

File: src/RobuROC_sim/src/description/RobuROC_core_vis.urdf.xacro (robot description, xacro)
@@ -43,11 +43,11 @@
     <!--                WHEEL 1  +x +y                   -->
     <!-- ##############################################  -->
-    <joint name="wheel_1_joint" type="continuous">
+    <joint name="wheel_1_joint" type="fixed">
         <origin xyz="${wheel_1_origin}" rpy="${-rot_90} 0 0"/>
         <parent link="base_link"/>
         <child link="wheel_1_link"/>
-        <axis xyz="0 0 1" />
+        <!-- <axis xyz="0 0 1" />
         <limit effort="1000" velocity="${max_vel}"/>
-        <dynamics damping="1.0" friction="1.0"/>
+        <dynamics damping="1.0" friction="1.0"/> -->
     </joint>
     <link name="wheel_1_link">
@@ -72,11 +72,11 @@
     <!--                WHEEL 2  +x -y                   -->
     <!-- ##############################################  -->
-    <joint name="wheel_2_joint" type="continuous">
+    <joint name="wheel_2_joint" type="fixed">
         <origin xyz="${wheel_2_origin}" rpy="${-rot_90} 0 0"/>
         <parent link="base_link"/>
         <child link="wheel_2_link"/>
-        <axis xyz="0 0 1" />
+        <!-- <axis xyz="0 0 1" />
         <limit effort="1000" velocity="${max_vel}"/>
-        <dynamics damping="1.0" friction="1.0"/>
+        <dynamics damping="1.0" friction="1.0"/> -->
     </joint>
     <link name="wheel_2_link">
@@ -101,11 +101,11 @@
     <!--                WHEEL 3  -x -y                   -->
     <!-- ##############################################  -->
-    <joint name="wheel_3_joint" type="continuous">
+    <joint name="wheel_3_joint" type="fixed">
         <origin xyz="${wheel_3_origin}" rpy="${-rot_90} 0 0"/>
         <parent link="base_link"/>
         <child link="wheel_3_link"/>
-        <axis xyz="0 0 1" />
+        <!-- <axis xyz="0 0 1" />
         <limit effort="1000" velocity="${max_vel}"/>
-        <dynamics damping="1.0" friction="1.0"/>
+        <dynamics damping="1.0" friction="1.0"/> -->
     </joint>
     <link name="wheel_3_link">
@@ -130,11 +130,11 @@
     <!--                WHEEL 4  -x +y                   -->
     <!-- ##############################################  -->
-    <joint name="wheel_4_joint" type="continuous">
+    <joint name="wheel_4_joint" type="fixed">
         <origin xyz="${wheel_4_origin}" rpy="${-rot_90} 0 0"/>
         <parent link="base_link"/>
         <child link="wheel_4_link"/>
-        <axis xyz="0 0 1" />
+        <!-- <axis xyz="0 0 1" />
         <limit effort="1000" velocity="${max_vel}"/>
-        <dynamics damping="1.0" friction="1.0"/>
+        <dynamics damping="1.0" friction="1.0"/> -->
     </joint>
     <link name="wheel_4_link">

File: src/RobuROC_sim/src/description/RobuROC_model.urdf.xacro (robot description, xacro)
@@ -4,5 +4,5 @@
     <xacro:include filename="include_RobuROC.xacro" />
     <!-- Add platform -->
-    <xacro:include filename="RobuROC_core.urdf.xacro" />
+    <xacro:include filename="RobuROC_core_vis.urdf.xacro" />
     <!-- Add two Realsense D435 RGB-D cameras -->
     <xacro:include filename="camera_depth.xacro"/>

File: src/RobuROC_sim/src/description/include_RobuROC.xacro (robot description, xacro)
@@ -37,9 +37,11 @@
     <xacro:property name="camera_off_x" value="0.6" />
     <xacro:property name="camera_off_z" value="0.55" />
-    <xacro:property name="camera_rot" value="${16*pi/180}" />
+    <xacro:property name="camera_rot" value="16" />
     <xacro:property name="camera_1_origin" value="${camera_off_x} 0 ${camera_off_z}" />
     <xacro:property name="camera_2_origin" value="${-camera_off_x} 0 ${camera_off_z}" />
-    <xacro:property name="camera_1_rotation" value="0 ${camera_rot} 0" />
-    <xacro:property name="camera_2_rotation" value="0 ${camera_rot} ${pi}" />
+    <!-- <xacro:property name="camera_2_origin" value="${camera_off_x-0.05} -0.32 ${camera_off_z}" /> -->
+    <xacro:property name="camera_1_rotation" value="0 ${(camera_rot)*pi/180} 0" />
+    <xacro:property name="camera_2_rotation" value="0 ${(camera_rot-2)*pi/180} ${pi}" />
+    <!-- <xacro:property name="camera_2_rotation" value="0 ${camera_rot} 0" /> -->
     <!-- ######################################### -->
     <!--                    Lidar                  -->
